File: Firmware/cc-pcb/cc-pcb/cc-pcb-1.27.sch (KiCad schematic (older format))
At the start: 16 parts, among them CON1 BARREL_JACK, IC1 ATMEGA328P-A, P1 CONN_20, P4 CONN_2, P5 CONN_6, P6 CONN_6, SW1 SRS

Commit message: Removed FreeRouting from the repo
Changed lines of the file:
@@
 Sheet 1 1
 Title "cc-schema.sch"
-Date "25 sep 2014"
+Date "30 sep 2014"
 Rev ""
 Comp ""
@@
 	5500 6000 5500 5550
 Wire Wire Line
-	5100 5100 8600 5100
-Wire Wire Line
-	5200 5000 8600 5000
-Wire Wire Line
-	5300 4900 8600 4900
-Wire Wire Line
-	5400 4800 8600 4800
-Wire Wire Line
-	5500 4700 8600 4700
-Wire Wire Line
-	5600 4600 8600 4600
-Wire Wire Line
-	5700 4500 8600 4500
-Wire Wire Line
-	5800 4400 8600 4400
-Wire Wire Line
-	5100 4300 5100 5100
-Wire Wire Line
 	4200 4300 5100 4300
 Wire Wire Line
-	5200 4200 5200 5000
-Wire Wire Line
 	4200 4200 5200 4200
 Wire Wire Line
-	5300 4100 5300 4900
-Wire Wire Line
 	4200 4100 5300 4100
 Wire Wire Line
-	5400 4000 5400 4800
+	5400 4000 5400 5000
 Wire Wire Line
 	4200 4000 5400 4000
 Wire Wire Line
-	5500 3900 5500 4700
+	5500 3900 5500 5100
 Wire Wire Line
 	4200 3900 5500 3900
 Wire Wire Line
-	5600 3800 5600 4600
+	5600 3800 5600 4900
 Connection ~ 4300 3700
 Wire Wire Line
-	5700 3700 5700 4500
-Wire Wire Line
-	5800 3600 5800 4400
+	5700 3700 5700 4700
+Wire Wire Line
+	5800 3600 5800 4500
 Wire Wire Line
 	4200 3600 5800 3600
@@
 	8100 2000 8100 2400
 Wire Wire Line
-	6900 3200 6900 3600
-Wire Wire Line
-	6900 3600 8600 3600
-Wire Wire Line
 	7200 3100 7200 3500
 Wire Wire Line
 	7200 3500 8600 3500
 Wire Wire Line
-	7500 3000 7500 3400
-Wire Wire Line
-	7500 3400 8600 3400
-Wire Wire Line
-	7800 2900 7800 3300
-Wire Wire Line
-	7800 3300 8600 3300
-Wire Wire Line
-	8100 2800 8100 3200
-Wire Wire Line
-	8100 3200 8600 3200
+	7800 2900 7800 3400
+Wire Wire Line
+	8100 2800 8100 3600
+Wire Wire Line
+	5800 4500 8600 4500
+Wire Wire Line
+	5700 4700 8600 4700
+Wire Wire Line
+	5600 4900 8600 4900
+Wire Wire Line
+	5500 5100 8600 5100
+Wire Wire Line
+	5400 5000 8600 5000
+Wire Wire Line
+	5300 4100 5300 4800
+Wire Wire Line
+	5300 4800 8600 4800
+Wire Wire Line
+	5200 4200 5200 4600
+Wire Wire Line
+	5200 4600 8600 4600
+Wire Wire Line
+	5100 4300 5100 4400
+Wire Wire Line
+	5100 4400 8600 4400
+Wire Wire Line
+	7500 3000 7500 3200
+Wire Wire Line
+	7500 3200 8600 3200
+Wire Wire Line
+	7800 3400 8600 3400
+Wire Wire Line
+	8100 3600 8600 3600
+Wire Wire Line
+	6900 3200 6900 3300
+Wire Wire Line
+	6900 3300 8600 3300
 $EndSCHEMATC

Commit message: First PCB
Changed lines of the file:
@@
 Sheet 1 1
 Title "cc-schema.sch"
-Date "30 sep 2014"
+Date "1 oct 2014"
 Rev ""
 Comp ""
@@
 	4200 3250 6000 3250
 Wire Wire Line
-	6000 3250 6000 4200
-Wire Wire Line
-	6000 4200 8600 4200
-Wire Wire Line
 	4200 3150 6100 3150
 Wire Wire Line
-	6100 3150 6100 4100
-Wire Wire Line
-	6100 4100 8600 4100
-Wire Wire Line
 	4200 3050 6200 3050
 Wire Wire Line
-	6200 3050 6200 4000
-Wire Wire Line
-	6200 4000 8600 4000
-Wire Wire Line
 	4200 2950 6300 2950
 Wire Wire Line
-	6300 2950 6300 3900
-Wire Wire Line
-	6300 3900 8600 3900
+	6300 2950 6300 4000
 Wire Wire Line
 	4200 2850 6400 2850
 Wire Wire Line
-	6400 2850 6400 3800
-Wire Wire Line
-	6400 3800 8600 3800
+	6400 2850 6400 4200
 Wire Wire Line
 	4200 2500 6600 2500
@@
 	8100 2000 8100 2400
 Wire Wire Line
-	7200 3100 7200 3500
-Wire Wire Line
-	7200 3500 8600 3500
-Wire Wire Line
 	7800 2900 7800 3400
 Wire Wire Line
@@
 	8100 3600 8600 3600
 Wire Wire Line
-	6900 3200 6900 3300
-Wire Wire Line
-	6900 3300 8600 3300
+	6000 3250 6000 4100
+Wire Wire Line
+	6000 4100 8600 4100
+Wire Wire Line
+	6100 3150 6100 3900
+Wire Wire Line
+	6100 3900 8600 3900
+Wire Wire Line
+	6200 3050 6200 3800
+Wire Wire Line
+	6200 3800 8600 3800
+Wire Wire Line
+	6300 4000 8600 4000
+Wire Wire Line
+	6400 4200 8600 4200
+Wire Wire Line
+	6900 3500 8600 3500
+Wire Wire Line
+	6900 3200 6900 3500
+Wire Wire Line
+	7200 3100 7200 3300
+Wire Wire Line
+	7200 3300 8600 3300
 $EndSCHEMATC

Commit message: in the middle of routing...
Parts:
- removed P5, P6: CONN_6, symbol CONN_6
- added P10, P11, P5, P6, P7, P8, P9: CONN_1, symbol CONN_1
- renumbered P4 to P2
Connections:
- wire segments 116 -> 107
Other:
- moved on the sheet: D1, D2, D3, D4, D5, D6

Commit message: in the middle of routing...
Connections:
- net at D4.1 (A): now also P1.7 (P7); no longer P1.11 (P11)
- net at D6.1 (A): now also P1.11 (P11); no longer P1.7 (P7)
Changed lines of the file:
@@
 Sheet 1 1
 Title "cc-schema.sch"
-Date "3 nov 2014"
+Date "4 nov 2014"
 Rev ""
 Comp ""
@@
 	6600 2500 6600 2800
 Wire Wire Line
-	6600 3200 6600 3800
+	6600 3200 6600 4200
 Wire Wire Line
 	4200 2400 6900 2400
@@
 Wire Wire Line
 	6900 3100 6900 4000
-Wire Wire Line
-	7200 3000 7200 4200
 $Comp
 L CONN_1 P7
@@
 $EndComp
 Wire Wire Line
-	6600 3800 8600 3800
-Wire Wire Line
 	6900 4000 8600 4000
 Wire Wire Line
-	7200 4200 8600 4200
-Wire Wire Line
 	6200 3050 6200 3700
 Wire Wire Line
@@
 Wire Wire Line
 	6400 3300 8600 3300
+Wire Wire Line
+	7200 3000 7200 3800
+Wire Wire Line
+	7200 3800 8600 3800
+Wire Wire Line
+	6600 4200 8600 4200
 $EndSCHEMATC

Commit message: finalizing pcb...
Parts:
- added P4: GND, symbol CONN_1
- P10: value CONN_1 -> SCK
- P11: value CONN_1 -> MISO
- P5: value CONN_1 -> DTR
- P6: value CONN_1 -> TXD
- P7: value CONN_1 -> RXD
- P8: value CONN_1 -> RST
- P9: value CONN_1 -> MOSI
Connections:
- net GND: now also P4.1
Other:
- moved on the sheet: C2, P10, P11, P5, P6, P7, P8, P9

Commit message: finalizing pcb...
Changed lines of the file:
@@
 	6900 2400 6900 2700
 Wire Wire Line
-	4200 2400 4800 2400
-Wire Wire Line
-	4800 2400 6900 2400
+	4200 2400 6900 2400
 Wire Wire Line
 	6600 3200 6600 4200
@@
 	6600 2500 6600 2800
 Wire Wire Line
-	4200 2500 4700 2500
-Wire Wire Line
-	4700 2500 6600 2500
+	4200 2500 6600 2500
 Wire Wire Line
 	4200 2850 6400 2850
@@
 	2200 2100 2300 2100
 Wire Wire Line
-	2200 1800 2200 2000
-Wire Wire Line
-	2200 2000 2200 2100
-Wire Wire Line
-	2200 2100 2200 2300
+	2200 1800 2200 2300
 Connection ~ 2700 1250
 Wire Wire Line
@@
 	4950 1000 4950 1200
 Wire Wire Line
-	4200 2300 4600 2300
-Wire Wire Line
-	4600 2300 7200 2300
+	4200 2300 7200 2300
 Wire Wire Line
 	4350 2700 4350 1000
@@
 	4300 3700 4300 5650
 Wire Wire Line
-	4200 3700 4300 3700
-Wire Wire Line
-	4300 3700 5700 3700
+	4200 3700 5700 3700
 Wire Wire Line
 	4400 5800 2800 5800
@@
 	2550 950  2700 950
 Wire Wire Line
-	2700 950  2700 1050
-Wire Wire Line
-	2700 1050 2700 1250
-Wire Wire Line
-	2700 1250 2700 1300
+	2700 950  2700 1300
 Wire Wire Line
 	2550 1050 2700 1050
@@
 	2700 850  2550 850
 Wire Wire Line
-	2700 700  2700 750
-Wire Wire Line
-	2700 750  2700 850
+	2700 700  2700 850
 Wire Wire Line
 	2200 2300 2300 2300
@@
 	3100 4750 3300 4750
 Wire Wire Line
-	3800 4750 3950 4750
+	3800 4750 4500 4750
 Wire Wire Line
-	3950 4750 4500 4750
-Wire Wire Line
-	4500 3450 4500 4750
-Wire Wire Line
-	4500 4750 4500 6000
+	4500 3450 4500 6000
 Wire Wire Line
 	4500 3450 4200 3450
@@
 Connection ~ 4600 2300
 Wire Wire Line
-	4200 3600 4400 3600
-Wire Wire Line
-	4400 3600 5800 3600
+	4200 3600 5800 3600
 Wire Wire Line
 	5800 3600 5800 4500
@@
 	2300 4100 2200 4100
 Wire Wire Line
-	2200 4100 2200 4200
-Wire Wire Line
-	2200 4200 2200 4300
-Wire Wire Line
-	2200 4300 2200 4450
+	2200 4100 2200 4450
 Wire Wire Line
 	2300 4200 2200 4200
